File: hardware/kicad/Communication_pcb_main.kicad_pcb (KiCad board)
At the start: 2 copper layers, 54 x 71 mm, 144 parts, among them J201 TYPE-C 16PIN 2MD(073), J202 WAFER-PH2.0-3PWB, J204 Conn_01x04, J205 Conn_01x02, J206 Conn_01x02, J401 Conn_01x04, J402 Conn_01x06, J403 Conn_01x02_Pin, J404 Conn_01x04, Q201 AO3400A, Q202 AO3400A, Q203 AO3400A, Q204 AO3400A, Q206 AO3400A, Q401 2N7002, Q402 2N7002, Q403 2N7002, Q404 AO3401A, Q405 2N7002, Q406 2N7002, Q407 AO3401A, SW603 TS-1088-AR02016, U202 BQ25792RQMR, U401 ZX-RF-1-Z21.25X, U402 ZX-RF-1-Z21.25X, U403 A7672E (LASE), U404 ESDBW5V0A1_C5173252, U405 ESP32-C6-MINI-1-N4, U406 SC7A20HTR, U602 GD25Q128ESIGR, U603 RT9080-33GJ5, U604 ATECC608B-SSHDA-T

Commit message: missed stuff
Parts:
- removed C216: 2.2uF, PCM_JLCPCB:C_0805
- removed C608: 22uF, PCM_JLCPCB:C_1206
- removed R215: 2.2Ω, PCM_JLCPCB:R_0805
- removed R652, R653, R698: 10kΩ, PCM_JLCPCB:R_0402
- added C416: 22uF, PCM_JLCPCB:C_0805, F.Cu at (123.0, 78.4)
- added C417: 1uF, PCM_JLCPCB:C_0603, F.Cu at (130.8, 130.1)
- added C418: 100pF, PCM_JLCPCB:C_0805, F.Cu at (154.7, 109.1)
- added C698: 100nF, PCM_JLCPCB:C_0402, F.Cu at (131.2, 92.7)
- added D403: ESD9X3.3ST5G, easyeda2kicad:SOD-923_L0.8-W0.6-LS1.0-RD, F.Cu at (161.4, 109.4)
- added D406: ESD9X3.3ST5G, easyeda2kicad:SOD-923_L0.8-W0.6-LS1.0-RD, F.Cu at (149.0, 69.3)
- added D407: 1N5819WS, easyeda2kicad:SOD-323_L1.8-W1.3-LS2.5-RD, F.Cu at (138.1, 83.8)
- added D420: Green, PCM_JLCPCB:D_0805, F.Cu at (126.7, 78.8)
- added G***: LOGO, LOGO, F.Cu at (149.0, 128.9)
- added G***: LOGO, LOGO, B.Cu at (143.4, 127.1)
- added G***: LOGO, LOGO, B.Cu at (161.7, 86.8)
- added G***: LOGO, LOGO, B.Cu at (144.9, 121.5)
- added H401: MountingHole, MountingHole:MountingHole_2.2mm_M2_ISO14580_Pad, F.Cu at (123.0, 124.1)
- added H402: MountingHole, weberel:Slot_2.2mm_M2_ISO14580_Pad, F.Cu at (157.0, 63.0)
- added H403: MountingHole, MountingHole:MountingHole_2.2mm_M2_ISO14580_Pad, F.Cu at (156.0, 136.1)
- added H404: MountingHole, weberel:Slot_2.2mm_M2_ISO14580_Pad, F.Cu at (168.1, 123.1)
- added L402: MPZ2012S221AT000, easyeda2kicad:L0805, F.Cu at (123.7, 128.8)
- added L403: GZ2012D601TF, easyeda2kicad:L0805, F.Cu at (126.2, 84.8)
- added L404: GZ2012D601TF, easyeda2kicad:L0805, F.Cu at (153.6, 106.8)
- added L407: RSCM7060-701, easyeda2kicad:FILTER-SMD_4P-L7.0-W6.0-P3.00-TL, F.Cu at (136.7, 133.7)
- added Q408: AO3400A, easyeda2kicad:SOT-23-3_L2.9-W1.3-P1.90-LS2.4-BR, F.Cu at (137.2, 79.4)
- added Q409: AO3400A, easyeda2kicad:SOT-23-3_L2.9-W1.3-P1.90-LS2.4-BR, F.Cu at (141.8, 75.4)
- added R422: 10kΩ, PCM_JLCPCB:R_0402, F.Cu at (139.6, 79.4)
- added R423: 10kΩ, PCM_JLCPCB:R_0402, F.Cu at (135.8, 77.8)
- added R424: 2.2Ω, PCM_JLCPCB:R_0603, F.Cu at (133.2, 128.8)
- added R425: 4.7kΩ, PCM_JLCPCB:R_0402, F.Cu at (138.6, 75.6)
- added R426: 47kΩ, PCM_JLCPCB:R_0402, F.Cu at (139.6, 76.2)
- added R427: 100kΩ, PCM_JLCPCB:R_0402, F.Cu at (125.6, 81.0)
- added R454: 100kΩ, PCM_JLCPCB:R_0402, F.Cu at (126.0, 77.1)
- added TP410: TestPoint, TestPoint:TestPoint_Pad_D1.0mm, B.Cu at (123.7, 71.7)
- added U407: LTR-303ALS-01, easyeda2kicad:TDFN-6_L2.0-W2.0-P0.65-BL, F.Cu at (132.9, 91.7)
- C401, C410: value 100uF -> 47uF; footprint PCM_JLCPCB:C_CASE-B-3528-21(mm) -> PCM_JLCPCB:C_1206
- D401: value SMAJ28A_C148227 -> SMAJ30A; footprint easyeda2kicad:SMA_L4.4-W2.8-LS5.4-RD -> easyeda2kicad:SMA_L4.3-W2.6-LS5.2-RD
- J204, J401, J404: footprint Connector_PinHeader_2.54mm:PinHeader_1x04_P2.54mm_Vertical -> weberel:custom_01x04_2.54
- J205, J206: footprint Connector_PinSocket_2.54mm:PinSocket_1x02_P2.54mm_Vertical -> weberel:custom_1x02_2.54
- J402: footprint Connector_PinHeader_2.54mm:PinHeader_1x06_P2.54mm_Vertical -> weberel:custom_01x06_2.54
- J403: footprint Connector_PinHeader_2.54mm:PinHeader_1x02_P2.54mm_Vertical -> weberel:custom_1x02_2.54
- Q401, Q402, Q403, Q405, Q406: value 2N7002 -> AO3400A; footprint PCM_JLCPCB:Q_SOT-23 -> easyeda2kicad:SOT-23-3_L2.9-W1.3-P1.90-LS2.4-BR
- R223: value 150kΩ -> 150Ω
- R418, R421: value 10kΩ -> 100kΩ
- moved C693 35.3 mm to (134.6, 114.7), turned to 90 degrees
- moved TP404 35.1 mm to (141.0, 81.3), turned to -90 degrees
- moved TP403 34.5 mm to (141.0, 83.8), turned to -90 degrees
- moved C697 34.2 mm to (135.7, 114.7), turned to -90 degrees
- moved J205 33.1 mm to (148.6, 134.6), turned to 90 degrees
- moved U406 32.4 mm to (137.8, 115.1), turned to 180 degrees
- moved C604 30.0 mm to (127.6, 118.3), turned to 180 degrees
- moved TP406 29.9 mm to (141.0, 78.7), turned to -90 degrees
- moved TP405 29.5 mm to (141.0, 76.2), turned to -90 degrees
- moved U604 28.6 mm to (129.3, 115.2)
- moved SW603 26.8 mm to (141.1, 70.8)
- moved C605 25.7 mm to (139.0, 73.0), turned to 0 degrees
- moved C606 25.6 mm to (141.0, 73.0), turned to 0 degrees
- moved R603 25.6 mm to (137.6, 75.2), turned to -90 degrees
- moved R604 24.5 mm to (139.4, 74.0), turned to 180 degrees
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Connections:
- C413 pad 1: Net-(U403-GNSS_ANT) -> Net-(D403-A)
- C414 pad 1: Net-(U403-GNSS_ANT) -> Net-(D403-A)
- C609 pad 2: /MCU/DN -> /MCU/DP
- C610 pad 2: /MCU/DP -> /MCU/DN
- D212 pad 5: /PowerManagament/VUSB -> Net-(D212-VBUS)
- D401 pad 1: /PowerManagament/Solar 5-20V -> Net-(D401-K)
- D401 pad 2: GND -> Net-(D401-A)
- D606 pad 5: /MCU/PWR -> Net-(D606-VBUS)
- J201 pad 11: /PowerManagament/VUSB -> Net-(D212-VBUS)
- J201 pad 2: /PowerManagament/VUSB -> Net-(D212-VBUS)
- J204 pad 2: /PowerManagament/VUSB -> Net-(D212-VBUS)
- J205 pad 1: GND -> Net-(D401-A)
- J205 pad 2: /PowerManagament/Solar 5-20V -> Net-(D401-K)
- J404 pad 2: /MCU/PWR -> Net-(D606-VBUS)
- R412 pad 1: Net-(U403-GNSS_ANT) -> Net-(D403-A)
- R412 pad 2: Net-(U403-GNSS_ANT) -> Net-(D403-A)
- R650 pad 1: /MCU/DN -> /MCU/DP
- R651 pad 1: /MCU/DP -> /MCU/DN
- U402 pad 1: Net-(U403-GNSS_ANT) -> Net-(D403-A)
- U403 pad 1: /MCU/PWRKEY -> Net-(Q409-D)
- U403 pad 66: unconnected-(U403-STATUS-Pad66) -> Net-(Q408-S)
- U403 pad 99: unconnected-(U403-VDD_AUX-Pad99) -> Net-(U403-VDD_AUX)
- U405 pad 10: Net-(U405-IO5) -> /MCU/SO
- U405 pad 12: /MCU/RX -> /MCU/STATUS
- U405 pad 13: /MCU/TX -> Net-(U405-IO1)
- U405 pad 20: Net-(U405-IO15) -> GND
- U405 pad 24: /MCU/SI -> /MCU/SCLK
- U405 pad 25: /MCU/SO -> /MCU/INT
- U405 pad 26: /MCU/SCLK -> /MCU/RX
- U405 pad 27: /MCU/INT -> /MCU/TX
- U405 pad 9: Net-(U405-IO4) -> /MCU/SI
- U406 pad 5: /MCU/INT_acc -> Net-(D407-K)
Routing:
- net /MCU/3V3_esp32: track 131.4 -> 37.2 mm, vias 2 -> 22
- net /MCU/INT: track 119.5 -> 63.5 mm, vias 14 -> 3
- net Net-(U403-VDD_AUX): track 0.00 -> 36.5 mm, vias 0 -> 2
- net Net-(D212-VBUS): track 0.00 -> 33.7 mm, vias 0 -> 3
- net Net-(D407-K): track 0.00 -> 30.6 mm
- net Net-(U405-IO13): track 30.2 -> 2.54 mm, vias 4 -> 0
- net Net-(U405-IO12): track 29.5 -> 2.44 mm, vias 4 -> 0
- net /MCU/VSYS: track 21.8 -> 0.00 mm, vias 24 -> 20
- net Net-(U403-GND-Pad91): track 0.00 -> 21.8 mm, vias 0 -> 4
- net /MCU/STATUS: track 0.00 -> 21.0 mm, vias 0 -> 2
- net /MCU/TX: track 40.8 -> 19.8 mm, vias 4 -> 0
- net /MCU/INT_acc: track 20.8 -> 41.5 mm, vias 5 -> 2
- net /MCU/RX: track 35.7 -> 16.5 mm, vias 4 -> 0
- net /MCU/PWRKEY: track 23.1 -> 6.19 mm, vias 6 -> 2
- net /MCU/QON: track 112.8 -> 96.5 mm, vias 12 -> 2
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- added copper zone on F.Cu, net /MCU/3V3_esp32
- added copper zone on In2.Cu, net /MCU/3V3_esp32
- added copper zone on In2.Cu, net /MCU/VSYS
- added copper zone on F.Cu, net /PowerManagament/REGN
- added copper zone on F.Cu, net /PowerManagament/VUSB
- added copper zone on In1.Cu, net GND
- added copper zone on F.Cu, net Net-(D212-VBUS)
- added copper zone on In2.Cu, net Net-(D212-VBUS)
- added copper zone on F.Cu, net Net-(D401-A)
- added copper zone on F.Cu, net Net-(D401-K)
- added copper zone on F.Cu, net Net-(D606-VBUS)
- removed copper zone on B.Cu, net /MCU/VSYS
Other:
- board size 54 x 71 mm -> 46 x 74 mm
- copper layers 2 -> 4
- board text added: "+ -"
- board text added: "10mm"
- board text added: "11mm"
- board text added: "14mm"
- board text added: "1mm"
- board text added: "2mm"
- board text added: "3V3"
- board text added: "46x74mm"
- board text added: "BOOT"
- board text added: "BTN"
- board text added: "CS"
- board text added: "DN"
- board text added: "DP"
- board text added: "GND"
- board text added: "GPIO 01"
- board text added: "QON"
- board text added: "RESET"
- board text added: "RX"
- board text added: "Rev A 23/04/2026"
- board text added: "SCL"
- board text added: "SCLK"
- board text added: "SDA"
- board text added: "SENSOR"
- board text added: "SI"
- board text added: "SO"
- board text added: "SPI"
- board text added: "TS"
- board text added: "TX"
- board text added: "USB"
- board text added: "VBAT"
- board text added: "VIN"
- board text added: "VSYS"
- board text added: "VUSB"
- board text added: "mr fancypants using wifi...."
- board text removed: "3A Solar/USB"
- board text removed: "E.Weber"
