File: hardware/kicad/Communication_pcb_main.kicad_sch (KiCad schematic)
At the start: 0 parts

Commit message: missed stuff
Parts:
- added H401, H403: MountingHole, MountingHole:MountingHole_2.2mm_M2_ISO14580_Pad, symbol Mechanical:MountingHole
- added H402, H404: MountingHole, weberel:Slot_2.2mm_M2_ISO14580_Pad, symbol Mechanical:MountingHole
Other:
- sheet MCU ports: added STATUS; removed none
- sheet SimCom ports: added STATUS; removed none
