File: hardware/kicad/mcu.kicad_sch (KiCad schematic)
At the start: 45 parts, among them J401 Conn_01x04, J402 Conn_01x06, J403 Conn_01x02_Pin, J404 Conn_01x04, Q405 2N7002, Q407 AO3401A, SW603 TS-1088-AR02016, U405 ESP32-C6-MINI-1-N4, U406 SC7A20HTR, U602 GD25Q128ESIGR, U603 RT9080-33GJ5, U604 ATECC608B-SSHDA-T

Commit message: missed stuff
Parts:
- removed C608: 22uF, PCM_JLCPCB:C_1206, symbol PCM_JLCPCB-Capacitors:1206,22uF
- removed Q405: 2N7002, PCM_JLCPCB:Q_SOT-23, symbol PCM_JLCPCB-Transistors:NMOS,2N7002
- removed R421, R652, R653, R698: 10kΩ, PCM_JLCPCB:R_0402, symbol PCM_JLCPCB-Resistors:0402,10kΩ
- added C416: 22uF, PCM_JLCPCB:C_0805, symbol PCM_JLCPCB-Capacitors:0805,22uF
- added C698: 100nF, PCM_JLCPCB:C_0402, symbol PCM_JLCPCB-Capacitors:0402,100nF
- added D407: 1N5819WS, easyeda2kicad:SOD-323_L1.8-W1.3-LS2.5-RD, symbol easyeda2kicad:1N5819WS
- added D420: Green, PCM_JLCPCB:D_0805, symbol PCM_JLCPCB-Diodes:LED,0805,Green
- added L403: GZ2012D601TF, easyeda2kicad:L0805, symbol easyeda2kicad:GZ2012D601TF
- added Q405: AO3400A, easyeda2kicad:SOT-23-3_L2.9-W1.3-P1.90-LS2.4-BR, symbol easyeda2kicad:AO3400A
- added R421, R427, R454: 100kΩ, PCM_JLCPCB:R_0402, symbol PCM_JLCPCB-Resistors:0402,100kΩ
- added TP410: TestPoint, TestPoint:TestPoint_Pad_D1.0mm, symbol Connector:TestPoint
- added U407: LTR-303ALS-01, easyeda2kicad:TDFN-6_L2.0-W2.0-P0.65-BL, symbol easyeda2kicad:LTR-303ALS-01
- J401, J404: footprint Connector_PinHeader_2.54mm:PinHeader_1x04_P2.54mm_Vertical -> weberel:custom_01x04_2.54; now left out of the parts list
- J402: footprint Connector_PinHeader_2.54mm:PinHeader_1x06_P2.54mm_Vertical -> weberel:custom_01x06_2.54; now left out of the parts list
- J403: footprint Connector_PinHeader_2.54mm:PinHeader_1x02_P2.54mm_Vertical -> weberel:custom_1x02_2.54
Connections:
- net 3V3_esp32: now also C416.2, C698.2, R427.1, U407.1 (VDD)
- net DN: now also C610.2, R651.1; no longer C609.2, R650.1
- net DP: now also C609.2, R650.1; no longer C610.2, R651.1
- net GND: now also U405.20 (IO15), C416.1, C698.1, D420.1, Q405.2 (S), U407.3 (GND)
- net INT: now also U405.25 (IO19); no longer U405.27 (IO21)
- net INT_acc: now also D407.2 (A), R427.2, U407.5 (INT); no longer U406.5 (INT1)
- net PWR: now also L403.1; no longer D606.5 (VBUS), J404.2 (Pin_2)
- net RX: now also U405.26 (IO20); no longer U405.12 (IO0)
- net SCL: now also U407.4 (SCL)
- net SCLK: now also U405.24 (IO18); no longer U405.26 (IO20)
- net SDA: now also U407.6 (SDA)
- net SI: now also U405.9 (IO4); no longer U405.24 (IO18)
- net SO: now also U405.10 (IO5); no longer U405.25 (IO19)
- net TX: now also U405.27 (IO21); no longer U405.13 (IO1)
- net VSYS: now also R421.2
- net at R419.2, R420.1: now also Q405.1 (G)
- net at Q407.1 (G): now also Q405.3 (D), R421.1
- new net: D407.1 (K), U406.5 (INT1)
- new net: D606.5 (VBUS), J404.2 (Pin_2), L403.2
- new net: D420.2, R454.2
- new net: R454.1, TP410.1, U405.13 (IO1)
- new net STATUS: U405.12 (IO0)
Other:
- moved on the sheet: D606, J401, J402, J404, R603, TP404
