File: hardware/kicad/power_mgmt.kicad_sch (KiCad schematic)
At the start: 52 parts, among them J201 TYPE-C 16PIN 2MD(073), J202 WAFER-PH2.0-3PWB, J204 Conn_01x04, J205 Conn_01x02, J206 Conn_01x02, Q201 AO3400A, Q202 AO3400A, Q203 AO3400A, Q204 AO3400A, Q206 AO3400A, U202 BQ25792RQMR

Commit message: missed stuff
Parts:
- removed C216: 2.2uF, PCM_JLCPCB:C_0805, symbol PCM_JLCPCB-Capacitors:0805,2.2uF
- removed D401: SMAJ28A_C148227, easyeda2kicad:SMA_L4.4-W2.8-LS5.4-RD, symbol easyeda2kicad:SMAJ28A_C148227
- removed R215: 2.2Ω, PCM_JLCPCB:R_0805, symbol PCM_JLCPCB-Resistors:0805,2.2Ω
- removed R223: 150kΩ, PCM_JLCPCB:R_0603, symbol PCM_JLCPCB-Resistors:0603,150kΩ
- added C417: 1uF, PCM_JLCPCB:C_0603, symbol PCM_JLCPCB-Capacitors:0603,1uF
- added D401: SMAJ30A, easyeda2kicad:SMA_L4.3-W2.6-LS5.2-RD, symbol easyeda2kicad:SMAJ30A
- added L402: MPZ2012S221AT000, easyeda2kicad:L0805, symbol easyeda2kicad:MPZ2012S221AT000
- added L407: RSCM7060-701, easyeda2kicad:FILTER-SMD_4P-L7.0-W6.0-P3.00-TL, symbol easyeda2kicad:RSCM7060-701
- added R223: 150Ω, PCM_JLCPCB:R_0603, symbol PCM_JLCPCB-Resistors:0603,150Ω
- added R424: 2.2Ω, PCM_JLCPCB:R_0603, symbol PCM_JLCPCB-Resistors:0603,2.2Ω
- J204: footprint Connector_PinHeader_2.54mm:PinHeader_1x04_P2.54mm_Vertical -> weberel:custom_01x04_2.54
- J205, J206: footprint Connector_PinSocket_2.54mm:PinSocket_1x02_P2.54mm_Vertical -> weberel:custom_1x02_2.54
Connections:
- net GND: now also C417.1, L407.4; no longer J205.1 (Pin_1)
- net Solar 5-20V: now also L407.3, R424.2; no longer J205.2 (Pin_2)
- net TS: now also R223.2
- net VUSB: now also L402.1; no longer D212.5 (VBUS), J201.11 (VBUS), J201.2 (VBUS), J204.2 (Pin_2)
- net at R222.2: now also R223.1
- new net: C417.2, R424.1
- new net: D401.1 (K), J205.2 (Pin_2), L407.2
- new net: D401.2 (A), J205.1 (Pin_1), L407.1
- new net: D212.5 (VBUS), J201.11 (VBUS), J201.2 (VBUS), J204.2 (Pin_2), L402.2
Other:
- note added: "needs to be 150ohm ...."
- moved on the sheet: J205
