File: hardware/kicad/simcom.kicad_sch (KiCad schematic)
At the start: 47 parts, among them Q401 2N7002, Q402 2N7002, Q403 2N7002, Q404 AO3401A, Q406 2N7002, U401 ZX-RF-1-Z21.25X, U402 ZX-RF-1-Z21.25X, U403 A7672E (LASE), U404 ESDBW5V0A1_C5173252

Commit message: missed stuff
Parts:
- removed C401, C410: 100uF, PCM_JLCPCB:C_CASE-B-3528-21(mm), symbol PCM_JLCPCB-Capacitors:CASE-B-3528-21(mm),100uF
- removed Q401, Q402, Q403, Q406: 2N7002, PCM_JLCPCB:Q_SOT-23, symbol PCM_JLCPCB-Transistors:NMOS,2N7002
- removed R418: 10kΩ, PCM_JLCPCB:R_0402, symbol PCM_JLCPCB-Resistors:0402,10kΩ
- added C401, C410: 47uF, PCM_JLCPCB:C_1206, symbol PCM_JLCPCB-Capacitors:1206,47uF
- added C418: 100pF, PCM_JLCPCB:C_0805, symbol PCM_JLCPCB-Capacitors:0805,100pF
- added D403, D406: ESD9X3.3ST5G, easyeda2kicad:SOD-923_L0.8-W0.6-LS1.0-RD, symbol easyeda2kicad:ESD9X3.3ST5G
- added L404: GZ2012D601TF, easyeda2kicad:L0805, symbol easyeda2kicad:GZ2012D601TF
- added Q401, Q402, Q403, Q406, Q408, Q409: AO3400A, easyeda2kicad:SOT-23-3_L2.9-W1.3-P1.90-LS2.4-BR, symbol easyeda2kicad:AO3400A
- added R418: 100kΩ, PCM_JLCPCB:R_0402, symbol PCM_JLCPCB-Resistors:0402,100kΩ
- added R422, R423: 10kΩ, PCM_JLCPCB:R_0402, symbol PCM_JLCPCB-Resistors:0402,10kΩ
- added R425: 4.7kΩ, PCM_JLCPCB:R_0402, symbol PCM_JLCPCB-Resistors:0402,4.7kΩ
- added R426: 47kΩ, PCM_JLCPCB:R_0402, symbol PCM_JLCPCB-Resistors:0402,47kΩ
Connections:
- net 3V3: now also R423.1
- net GND: now also C401.2, C410.2, D403.1 (C), D406.1 (C), Q401.2 (S), Q406.2 (S), Q409.2 (S), R426.1
- net PWRKEY: now also R425.2; no longer U403.1 (PWRKEY)
- net RX: now also Q402.3 (D)
- net TX: now also Q403.3 (D)
- net VDD_1V8: now also Q402.1 (G), Q403.1 (G), Q408.1 (G), R422.2
- net VSYS: now also R418.2
- net Vin: now also C401.1, C410.1
- net at C413.1, C414.1, R412.1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: now also C418.1, D403.2 (A), L404.1; no longer U403.90 (GNSS_ANT)
- net at R402.2, R403.2: now also Q406.1 (G)
- net at R416.2, R417.1: now also Q401.1 (G)
- net at R407.1, U403.9 (TXD): now also Q403.2 (S)
- net at Q404.1 (G): now also Q401.3 (D), R418.1
- net at R404.2: now also Q406.3 (D)
- net at C405.1, C412.1, R401.1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: now also D406.2 (A)
- net at R406.2, U403.10 (RXD): now also Q402.2 (S)
- net at U403.66 (STATUS): now also Q408.2 (S), R422.1
- net at U403.99 (VDD_AUX): now also L404.2
- new net: Q409.1 (G), R425.1, R426.2
- new net: C418.2, U403.90 (GNSS_ANT)
- new net: Q409.3 (D), U403.1 (PWRKEY)
- new net STATUS: Q408.3 (D), R423.2
